Commit message: add lidar sim

File: src/jackal_description/urdf/custom.xacro (robot description, xacro)
@@ -1,11 +1,38 @@
 <?xml version="1.0"?>
 <robot xmlns:xacro="http://www.ros.org/wiki/xacro">
-    <!-- kinect -->
-    <xacro:include filename="$(find jackal_description)/urdf/sensors/kinect.xacro" />
-    <joint name="kinect_joint" type="fixed">
-        <origin xyz="0.05 0 0.02" rpy="0 0 0" />
-        <parent link="front_mount"/>
-        <child link="kinect_link"/>
-    </joint>
-    <xacro:kinect_camera prefix="kinect"/>
+  <!-- kinect -->
+  <xacro:include filename="$(find jackal_description)/urdf/sensors/kinect.xacro" />
+  <joint name="kinect_joint" type="fixed">
+    <origin xyz="0.05 0 0.02" rpy="0 0 0" />
+    <parent link="front_mount"/>
+    <child link="kinect_link"/>
+  </joint>
+  <xacro:kinect_camera prefix="kinect"/>
+  <!-- lidar tower -->
+  <link name="lidar_tower">
+    <visual>
+      <origin xyz="0 0 0" rpy="0 0 0"/>
+      <geometry>
+        <mesh filename="package://jackal_description/meshes/velodyne_tower.stl"/>
+      </geometry>
+      <material name="light_grey" />
+    </visual>
+  </link>
+  <gazebo reference="lidar_tower">
+    <material>Gazebo/LightGrey</material>
+    <turnGravityOff>false</turnGravityOff>
+  </gazebo>
+  <joint name="lidar_tower_joint" type="fixed">
+    <origin xyz="0 0 0" rpy="0 0 0" />
+    <parent link="mid_mount"/>
+    <child link="lidar_tower"/>
+  </joint>
+  <!-- lidar -->
+  <xacro:include filename="$(find jackal_description)/urdf/sensors/lidar.xacro" />
+  <joint name="lidar_joint" type="fixed">
+    <origin xyz="0 0 0.115" rpy="0 0 0" />
+    <parent link="lidar_tower"/>
+    <child link="laser_link"/>
+  </joint>
+  <xacro:rplidar prefix="laser"/>
 </robot>
