Commit message: add imu sim

File: src/jackal_description/urdf/jackal.urdf.xacro (robot description, xacro)
@@ -185,19 +185,4 @@
     <child link="imu_link" />
   </joint>
-  <!-- Default NAVSAT Link -->
-  <link name="navsat_link">
-    <visual>
-      <geometry>
-        <cylinder radius="0.026" length="0.016" />
-      </geometry>
-      <origin xyz="0 0 0.008" />
-      <material name="black" />
-    </visual>
-  </link>
-  <joint name="navsat_joint" type="fixed">
-    <parent link="chassis_link" />
-    <child link="navsat_link" />
-    <origin xyz="-0.180 0.126 0.1815" />
-  </joint>
   <link name="mid_mount"></link>
   <joint name="mid_mount_joint" type="fixed">
