Commit message: add gmapping

File: src/jackal_description/urdf/sensors/kinect.xacro (robot description, xacro)
@@ -1,5 +1,4 @@
 <?xml version="1.0"?>
 <robot xmlns:xacro="http://www.ros.org/wiki/xacro" name="kinect_camera">
-    <xacro:property name="M_PI" value="3.1415926"/>
     <xacro:macro name="kinect_camera" params="prefix:=camera">
         <!-- Create kinect reference frame -->
@@ -8,5 +7,5 @@
             <origin xyz="0 0 0" rpy="0 0 0"/>
             <visual>
-                <origin xyz="0 0 0" rpy="0 0 ${M_PI/2}"/>
+                <origin xyz="0 0 0" rpy="0 0 ${PI/2}"/>
                 <geometry>
                     <mesh filename="package://jackal_description/meshes/kinect/kinect.dae" />
@@ -30,5 +29,5 @@
                 <update_rate>20.0</update_rate>
                 <camera>
-                    <horizontal_fov>${60.0*M_PI/180.0}</horizontal_fov>
+                    <horizontal_fov>${60.0*PI/180.0}</horizontal_fov>
                     <image>
                         <format>R8G8B8</format>

File: src/jackal_description/urdf/sensors/lidar.xacro (robot description, xacro)
@@ -26,18 +26,24 @@
                     <scan>
                       <horizontal>
-                        <samples>360</samples>
-                        <resolution>1</resolution>
-                        <min_angle>-3</min_angle>
-                        <max_angle>3</max_angle>
+                        <!-- 总共有多少激光点 -->
+                        <samples>720</samples>
+                        <!-- 扫描范围（弧度），这里为360度 -->
+                        <min_angle>-${PI}</min_angle>
+                        <max_angle>${PI}</max_angle>
                       </horizontal>
                     </scan>
                     <range>
+                      <!-- 最近&最远距离，该范围外的物体不可见 -->
                       <min>0.10</min>
-                      <max>6.0</max>
+                      <max>5.0</max>
+                      <!-- 距离分辨率（精度），这里为1cm -->
                       <resolution>0.01</resolution>
                     </range>
                     <noise>
+                      <!-- 高斯噪声 -->
                       <type>gaussian</type>
+                      <!-- 均值 -->
                       <mean>0.0</mean>
+                      <!-- 标准差 -->
                       <stddev>0.01</stddev>
                     </noise>
